File: KiCad/SelfBalancingRobot/SelfBalancingRobot.kicad_sch (KiCad schematic)
At the start: 2 parts, among them U1 ESP32_NODEMCU, U2 GY-521

Commit message: kicad parts
Parts:
- added TB1: POLOLU-713, SHIELD_POLOLU-713, symbol POLOLU-713:POLOLU-713
- added U3, U4: ~, symbol 0_Library:V-TecMotorHeader
Connections:
- new net: TB1.1 (GND), TB1.8 (GND), TB1.9 (GND)
Other:
- moved on the sheet: U2
Changed lines of the file:
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@@
 (kicad_sch (version 20230121) (generator eeschema)
   (paper "A4")
+  (symbol (lib_id "0_Library:V-TecMotorHeader") (at 63.5 78.74 0) (unit 1)
+    (in_bom yes) (on_board yes) (dnp no) (fields_autoplaced)
+    (property "Reference" "U4" (at 69.85 79.375 0)
+      (effects (font (size 1.27 1.27)) (justify left))
+    )
+    (property "Value" "~" (at 60.96 77.47 0)
+      (effects (font (size 1.27 1.27)))
+    )
+    (property "Footprint" "" (at 60.96 77.47 0)
+      (effects (font (size 1.27 1.27)) hide)
+    )
+    (property "Datasheet" "" (at 60.96 77.47 0)
+      (effects (font (size 1.27 1.27)) hide)
+    )
+    (pin "1")
+    (pin "2")
+    (pin "3")
+    (pin "4")
+    (pin "5")
+    (pin "6")
+    (instances
+      (project "SelfBalancingRobot"
+        (path "/043c0707-b174-4524-b691-8cb08d8870c2"
+          (reference "U4") (unit 1)
+        )
+      )
+    )
+  )
   (symbol (lib_id "ESP32_NODEMCU:ESP32_NODEMCU") (at 135.89 95.25 0) (unit 1)
     (in_bom yes) (on_board yes) (dnp no) (fields_autoplaced)
@@
     )
   )
-  (symbol (lib_id "GY-521:GY-521") (at 218.44 93.98 0) (unit 1)
+  (symbol (lib_id "POLOLU-713:POLOLU-713") (at 229.87 119.38 0) (unit 1)
     (in_bom yes) (on_board yes) (dnp no) (fields_autoplaced)
-    (property "Reference" "U2" (at 237.49 95.885 0)
+    (property "Reference" "TB1" (at 229.87 100.33 0)
+      (effects (font (size 1.27 1.27)))
+    )
+    (property "Value" "POLOLU-713" (at 229.87 102.87 0)
+      (effects (font (size 1.27 1.27)))
+    )
+    (property "Footprint" "SHIELD_POLOLU-713" (at 229.87 119.38 0)
+      (effects (font (size 1.27 1.27)) (justify bottom) hide)
+    )
+    (property "Datasheet" "" (at 229.87 119.38 0)
+      (effects (font (size 1.27 1.27)) hide)
+    )
+    (property "STANDARD" "Manufacturer recommendations" (at 229.87 119.38 0)
+      (effects (font (size 1.27 1.27)) (justify bottom) hide)
+    )
+    (property "PARTREV" "" (at 229.87 119.38 0)
+      (effects (font (size 1.27 1.27)) (justify bottom) hide)
+    )
+    (property "MANUFACTURER" "POLOLU" (at 229.87 119.38 0)
+      (effects (font (size 1.27 1.27)) (justify bottom) hide)
+    )
+    (pin "1")
+    (pin "10")
+    (pin "11")
+    (pin "12")
+    (pin "13")
+    (pin "14")
+    (pin "15")
+    (pin "16")
+    (pin "2")
+    (pin "3")
+    (pin "4")
+    (pin "5")
+    (pin "6")
+    (pin "7")
+    (pin "8")
+    (pin "9")
+    (instances
+      (project "SelfBalancingRobot"
+        (path "/043c0707-b174-4524-b691-8cb08d8870c2"
+          (reference "TB1") (unit 1)
+        )
+      )
+    )
+  )
+  (symbol (lib_id "0_Library:V-TecMotorHeader") (at 63.5 44.45 0) (unit 1)
+    (in_bom yes) (on_board yes) (dnp no) (fields_autoplaced)
+    (property "Reference" "U3" (at 69.85 45.085 0)
       (effects (font (size 1.27 1.27)) (justify left))
     )
-    (property "Value" "GY-521" (at 237.49 98.425 0)
+    (property "Value" "~" (at 60.96 43.18 0)
+      (effects (font (size 1.27 1.27)))
+    )
+    (property "Footprint" "" (at 60.96 43.18 0)
+      (effects (font (size 1.27 1.27)) hide)
+    )
+    (property "Datasheet" "" (at 60.96 43.18 0)
+      (effects (font (size 1.27 1.27)) hide)
+    )
+    (pin "1")
+    (pin "2")
+    (pin "3")
+    (pin "4")
+    (pin "5")
+    (pin "6")
+    (instances
+      (project "SelfBalancingRobot"
+        (path "/043c0707-b174-4524-b691-8cb08d8870c2"
+          (reference "U3") (unit 1)
+        )
+      )
+    )
+  )
+  (symbol (lib_id "GY-521:GY-521") (at 222.25 63.5 0) (unit 1)
+    (in_bom yes) (on_board yes) (dnp no) (fields_autoplaced)
+    (property "Reference" "U2" (at 241.3 65.405 0)
       (effects (font (size 1.27 1.27)) (justify left))
     )
-    (property "Footprint" "GY-521" (at 218.44 93.98 0)
+    (property "Value" "GY-521" (at 241.3 67.945 0)
+      (effects (font (size 1.27 1.27)) (justify left))
+    )
+    (property "Footprint" "GY-521" (at 222.25 63.5 0)
       (effects (font (size 1.27 1.27)) (justify bottom) hide)
     )
-    (property "Datasheet" "" (at 218.44 93.98 0)
+    (property "Datasheet" "" (at 222.25 63.5 0)
       (effects (font (size 1.27 1.27)) hide)
     )

Commit message: kicad
Parts:
- removed U2: GY-521, GY-521, symbol GY-521:GY-521
- added C1, C2: C, Capacitor_THT:C_Disc_D6.0mm_W4.4mm_P5.00mm, symbol Device:C
- added C3, C4: C, Capacitor_THT:CP_Radial_D6.3mm_P2.50mm, symbol Device:C
- added H1, H2, H3, H4: MountingHole, MountingHole:MountingHole_3.2mm_M3_DIN965_Pad_TopBottom, symbol Mechanical:MountingHole
- added R1: 10kR, Resistor_THT:R_Axial_DIN0204_L3.6mm_D1.6mm_P7.62mm_Horizontal, symbol Device:R
- added U5: ~, 0_Footprints:BatteryConnector, symbol 0_Library:BatteryConnector
- added U6: ~, 0_Footprints:MPU-6050-External, symbol 0_Library:MPU-6050
- added U7: ~, 0_Footprints:CurrentMeter, symbol 0_Library:CurrentMeter
- added U8: L7805, Package_TO_SOT_THT:TO-220-3_Horizontal_TabDown, symbol Regulator_Linear:L7805
- U3, U4: footprint (none) -> 0_Footprints:V-TecMotorHeader
Connections:
- net at U4.1 (M1): now also TB1.5 (BO2), C2.1
- net at U4.2 (M2): now also TB1.6 (BO1), C2.2
- net +3.3V: now reaches U4.3 (VccEnc)
- net +3.3V: now also TB1.2 (VCC), U1.J5_19 (3V3), U3.3 (VccEnc), R1.1, U6.VCC
- net RPM-Right: now reaches U4.4 (Enc1)
- net RPM-Right: now also U1.J5_16 (I_39)
- net 0: now reaches U4.6 (EncGnd)
- net 0: now also TB1.1 (GND), TB1.8 (GND), TB1.9 (GND), U1.J4_1 (GND_J4_1), U1.J4_7 (GND_J4_7), U1.J5_6 (GND_J5_6), U3.6 (EncGnd), C3.2, C4.2, U5.GND, U6.GND, U7.1 (GND), U8.2 (GND)
- net Lmotor-PWM: now reaches U1.J4_10 (G5)
- net Lmotor-PWM: now also TB1.16 (PWMA)
- net Rmotor-1: now reaches U1.J4_11 (G17)
- net Rmotor-1: now also TB1.12 (BIN1)
- net Rmotor-2: now reaches U1.J4_12 (G16)
- net Rmotor-2: now also TB1.11 (BIN2)
- net Rmotor-PWM: now reaches U1.J4_13 (G4)
- net Rmotor-PWM: now also TB1.10 (PWMB)
- net LED-Internal: now reaches U1.J4_15 (G2)
- net MPU-INT: now reaches U1.J4_2 (G23)
- net MPU-INT: now also U6.INT
- net MPU-SCL: now reaches U1.J4_3 (G22)
- net MPU-SCL: now also U6.SCL
- net MPU-SDA: now reaches U1.J4_6 (G21)
- net MPU-SDA: now also U6.SDA
- net Lmotor-1: now reaches U1.J4_8 (G19)
- net Lmotor-1: now also TB1.14 (AIN1)
- net Lmotor-2: now reaches U1.J4_9 (G18)
- net Lmotor-2: now also TB1.15 (AIN2)
- net +5V: now reaches U1.J5_1 (5V)
- net +5V: now also C3.1, U7.3 (Vcc), U8.3 (OUT)
- net CurrentMeas: now reaches U1.J5_14 (G35)
- net CurrentMeas: now also U7.2 (Ival)
- net RPM-Left: now reaches U1.J5_17 (I_36)
- net RPM-Left: now also U3.4 (Enc1)
- net at TB1.13 (~{STBY}): now also R1.2
- net at TB1.3 (AO1): now also U3.1 (M1), C1.1
- net at TB1.4 (AO2): now also U3.2 (M2), C1.2
- net +BATT: now reaches TB1.7 (VMOT)
- net +BATT: now also C4.1, U7.p2 (Pout), U8.1 (IN)
- new net: U5.Vbatt, U7.p1 (Pin)
Other:
- moved on the sheet: U3, U4

Commit message: kicad layout finished1
Parts:
- removed R1: 10kR, Resistor_THT:R_Axial_DIN0204_L3.6mm_D1.6mm_P7.62mm_Horizontal, symbol Device:R
Connections:
- net MotorENABLE: now reaches U1.J5_9 (G27)
- net MotorENABLE: now also TB1.13 (~{STBY})
Changed lines of the file:
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@@
-    (stroke (width 0) (type default))
-  )
-  (wire (pts (xy 190.5 78.74) (xy 191.77 78.74))
     (stroke (width 0) (type default))
   )
@@
     )
   )
+  (global_label "MotorENABLE" (shape bidirectional) (at 156.21 105.41 0) (fields_autoplaced)
+    (effects (font (size 1.27 1.27)) (justify left))
+    (property "Intersheetrefs" "${INTERSHEET_REFS}" (at 172.5036 105.41 0)
+      (effects (font (size 1.27 1.27)) (justify left) hide)
+    )
+  )
   (global_label "Rmotor-2" (shape bidirectional) (at 156.21 82.55 0) (fields_autoplaced)
     (effects (font (size 1.27 1.27)) (justify left))
@@
     )
   )
-  (global_label "CurrentMeas" (shape input) (at 156.21 115.57 0) (fields_autoplaced)
-    (effects (font (size 1.27 1.27)) (justify left))
-    (property "Intersheetrefs" "${INTERSHEET_REFS}" (at 170.7876 115.57 0)
+  (global_label "CurrentMeas" (shape bidirectional) (at 156.21 115.57 0) (fields_autoplaced)
+    (effects (font (size 1.27 1.27)) (justify left))
+    (property "Intersheetrefs" "${INTERSHEET_REFS}" (at 171.8989 115.57 0)
       (effects (font (size 1.27 1.27)) (justify left) hide)
     )
@@
     )
   )
+  (global_label "MotorENABLE" (shape bidirectional) (at 199.39 78.74 180) (fields_autoplaced)
+    (effects (font (size 1.27 1.27)) (justify right))
+    (property "Intersheetrefs" "${INTERSHEET_REFS}" (at 183.0964 78.74 0)
+      (effects (font (size 1.27 1.27)) (justify right) hide)
+    )
+  )
   (global_label "MPU-SCL" (shape bidirectional) (at 156.21 95.25 0) (fields_autoplaced)
     (effects (font (size 1.27 1.27)) (justify left))
@@
     )
   )
-  (global_label "CurrentMeas" (shape input) (at 74.93 45.72 0) (fields_autoplaced)
-    (effects (font (size 1.27 1.27)) (justify left))
-    (property "Intersheetrefs" "${INTERSHEET_REFS}" (at 89.5076 45.72 0)
+  (global_label "CurrentMeas" (shape bidirectional) (at 74.93 45.72 0) (fields_autoplaced)
+    (effects (font (size 1.27 1.27)) (justify left))
+    (property "Intersheetrefs" "${INTERSHEET_REFS}" (at 90.6189 45.72 0)
       (effects (font (size 1.27 1.27)) (justify left) hide)
     )
@@
     )
   )
-  (symbol (lib_id "power:+3.3V") (at 190.5 78.74 0) (unit 1)
-    (in_bom yes) (on_board yes) (dnp no) (fields_autoplaced)
-    (property "Reference" "#PWR04" (at 190.5 82.55 0)
-      (effects (font (size 1.27 1.27)) hide)
-    )
-    (property "Value" "+3.3V" (at 190.5 74.93 0)
-      (effects (font (size 1.27 1.27)))
-    )
-    (property "Footprint" "" (at 190.5 78.74 0)
-      (effects (font (size 1.27 1.27)) hide)
-    )
-    (property "Datasheet" "" (at 190.5 78.74 0)
-      (effects (font (size 1.27 1.27)) hide)
-    )
-    (pin "1")
-    (instances
-      (project "SelfBalancingRobot"
-        (path "/043c0707-b174-4524-b691-8cb08d8870c2"
-          (reference "#PWR04") (unit 1)
-        )
-      )
-    )
-  )
   (symbol (lib_id "Device:C") (at 233.68 77.47 0) (unit 1)
     (in_bom yes) (on_board yes) (dnp no) (fields_autoplaced)
@@
         )
       )
-    )
-  )
-  (symbol (lib_id "Device:R") (at 195.58 78.74 90) (unit 1)
-    (in_bom yes) (on_board yes) (dnp no) (fields_autoplaced)
-    (property "Reference" "R1" (at 195.58 73.66 90)
-      (effects (font (size 1.27 1.27)))
-    )
-    (property "Value" "10kR" (at 195.58 76.2 90)
-      (effects (font (size 1.27 1.27)))
-    )
-    (property "Footprint" "Resistor_THT:R_Axial_DIN0204_L3.6mm_D1.6mm_P7.62mm_Horizontal" (at 195.58 80.518 90)
-      (effects (font (size 1.27 1.27)) hide)
-    )
-    (property "Datasheet" "~" (at 195.58 78.74 0)
-      (effects (font (size 1.27 1.27)) hide)
-    )
-    (pin "1")
-    (pin "2")
-    (instances
-      (project "SelfBalancingRobot"
-        (path "/043c0707-b174-4524-b691-8cb08d8870c2"
-          (reference "R1") (unit 1)
-        )
-      )

Commit message: kicad done and pid integrated
Parts:
- added ChargingConnector1: ~, 0_Footprints:ChargingConnector, symbol 0_Library:BatteryConnector
- added R1: 10k, Resistor_THT:R_Axial_DIN0207_L6.3mm_D2.5mm_P7.62mm_Horizontal, symbol Device:R
- added R2: 20k, Resistor_THT:R_Axial_DIN0207_L6.3mm_D2.5mm_P7.62mm_Horizontal, symbol Device:R
- added SW1: Charging Switch, Connector_Phoenix_MSTB:PhoenixContact_MSTBA_2,5_3-G-5,08_1x03_P5.08mm_Horizontal, symbol Switch:SW_SPDT
- C1, C2: value C -> 1uF
Connections:
- net 0: now also ChargingConnector1.GND, R2.2
- net CurrentMeas: now also R1.1, R2.1; no longer U7.2 (Ival)
- net at U5.Vbatt: now also SW1.2 (B); no longer U7.p1 (Pin)
- new net: R1.2, U7.2 (Ival)
- new net: ChargingConnector1.Vbatt, SW1.1 (A)
- new net: SW1.3 (C), U7.p1 (Pin)
Other:
- moved on the sheet: C1, C2, C3, C4, TB1, U3, U4, U5, U6, U7, U8
